File: WioTerminal_M5Adapter.kicad_pcb (KiCad board)
At the start: 2 copper layers, 68 x 52.5 mm, 50 parts, among them J1 Raspberry_Pi_2_3, J2 Ext. BAT, J3 GROVE, J4 GROVE, J5 MBUS_BOTTOM, J6 Ext. BAT, SW1 JS102011JAQN, U1 INA219, U2 TPS63060, U3 ATECC608A

Commit message: Fix INA-219 pin assignment
Parts:
- MH1, MH2, MH3, MH4: footprint local:MountingHole_2.2mm_M2_DIN965_Mask -> MountingHole:MountingHole_2.2mm_M2_DIN965
- MH5, MH6: footprint MountingHole:MountingHole_2.2mm_M2_DIN965 -> MountingHole:MountingHole_3.2mm_M3
- U1: value INA219 -> INA219AIDCN
- moved C2 6.07 mm to (35.5, -4.85), turned to 180 degrees
- moved U1 1.95 mm to (37.4, -7.23), turned to 0 degrees
Connections:
- J1 pad 18: (no net) -> Net-(J1-Pad18)
- J1 pad 22: (no net) -> Net-(J1-Pad22)
- J1 pad 29: (no net) -> Net-(J1-Pad29)
- J1 pad 36: (no net) -> Net-(J1-Pad36)
- J1 pad 37: (no net) -> Net-(J1-Pad37)
- J1 pad 7: (no net) -> Net-(J1-Pad7)
- J5 pad 30: (no net) -> /BATTERY
- J5 pad 6: (no net) -> Net-(J5-Pad6)
- U1 pad 1: /A1 -> Net-(F1-Pad1)
- U1 pad 2: /A0 -> Net-(C1-Pad1)
- U1 pad 3: /SDA -> GND
- U1 pad 4: /SCL -> +3V3
- U1 pad 5: +3V3 -> /SCL
- U1 pad 6: GND -> /SDA
- U1 pad 7: Net-(C1-Pad1) -> /A0
- U1 pad 8: Net-(F1-Pad1) -> /A1
- U3 pad 1: (no net) -> Net-(U3-Pad1)
- U3 pad 2: (no net) -> Net-(U3-Pad2)
- U3 pad 3: (no net) -> Net-(U3-Pad3)
- U3 pad 5: /SCL -> /SDA
- U3 pad 6: /SDA -> /SCL
- U3 pad 7: (no net) -> Net-(U3-Pad7)
Routing:
- net /SDA: track 69.3 -> 75.8 mm
- net /SCL: track 61.0 -> 66.5 mm
- net Net-(C1-Pad1): track 35.2 -> 39.1 mm
- net /A0: track 7.79 -> 11.1 mm, vias 0 -> 2
- net +3V3: track 86.9 -> 89.9 mm, vias 6 -> 7
- net /A1: track 5.32 -> 7.57 mm, vias 0 -> 2
- net Net-(R15-Pad2): track 30.1 -> 31.0 mm
- net GND: track 45.3 -> 45.4 mm, vias 116 -> 139
Other:
- board text added: "M5 Bottom Adapter for Wio Terminal 2020-07-19 Rev.B by Kenta IDA (@ciniml)"
- board text removed: "M5 Bottom Adapter for Wio Terminal 2020-06-15 Rev.A by Kenta IDA (@ciniml)"

Commit message: Add NMT jumper between MBUS +5V and BAT.
Parts:
- added R16: DNP, Resistor_SMD:R_0603_1608Metric, B.Cu at (47.1, -8.45)
Connections:
- J1 pad 18: Net-(J1-Pad18) -> (no net)
- J1 pad 22: Net-(J1-Pad22) -> (no net)
- J1 pad 29: Net-(J1-Pad29) -> (no net)
- J1 pad 36: Net-(J1-Pad36) -> (no net)
- J1 pad 37: Net-(J1-Pad37) -> (no net)
- J1 pad 7: Net-(J1-Pad7) -> (no net)
- J5 pad 6: Net-(J5-Pad6) -> (no net)
- U3 pad 1: Net-(U3-Pad1) -> (no net)
- U3 pad 2: Net-(U3-Pad2) -> (no net)
- U3 pad 3: Net-(U3-Pad3) -> (no net)
- U3 pad 7: Net-(U3-Pad7) -> (no net)
Routing:
- net +5V: track 98.8 -> 102.7 mm
- net /BATTERY: track 0.00 -> 2.65 mm
- net GND: vias 139 -> 137
